Commit message: fix(urdf): the whole urdf was rotated

File: src/bb_description/urdf/beuzebot.urdf (robot description, URDF)
Before this commit: robot beuzebot, 6 links, 4 joints
Links:
- link base_link: geometry visual box size=${BASE_LINK_DEPTH} ${BASE_LINK_WIDTH} ${BASE_LINK_HEIGHT}
Joints:
- joint base_to_lwheel: axis 0 0 1 -> 0 1 0; origin xyz=${BASE_LINK_TO_WHEEL_X} ${BASE_LINK_TO_WHEEL_Y} ${BASE_LINK_TO_WHEEL_Z} rpy=0 ${PI/2} 0 -> xyz=${BASE_LINK_TO_WHEEL_X} ${BASE_LINK_TO_WHEEL_Y} ${BASE_LINK_TO_WHEEL_Z} rpy=0 0 0
- joint base_to_rwheel: axis 0 0 1 -> 0 1 0; origin xyz=${-BASE_LINK_TO_WHEEL_X - WHEEL_LENGTH/2} ${BASE_LINK_TO_WHEEL_Y} ${BASE_LINK_TO_WHEEL_Z} rpy=0 ${PI/2} 0 -> xyz=${BASE_LINK_TO_WHEEL_X} ${-BASE_LINK_TO_WHEEL_Y - WHEEL_LENGTH/2} ${BASE_LINK_TO_WHEEL_Z} rpy=0 0 0
- joint caster_part_to_caster_wheel: axis 0 0 1 -> 0 1 0; origin xyz=${CASTER_PART_TO_CASTER_WHEEL_X} ${CASTER_PART_TO_CASTER_WHEEL_Y} ${CASTER_PART_TO_CASTER_WHEEL_Z} rpy=0 ${PI/2} 0 -> xyz=${CASTER_PART_TO_CASTER_WHEEL_X} ${CASTER_PART_TO_CASTER_WHEEL_Y} ${CASTER_PART_TO_CASTER_WHEEL_Z} rpy=0 0 0

Commit message: fix(odom): publish odom by reference to middle wheel

File: src/bb_description/urdf/beuzebot.urdf (robot description, URDF)
Before this commit: robot beuzebot, 6 links, 4 joints
Links:
- added link middle_wheel
Joints:
- added joint middle_wheel_to_base: type continuous, parent middle_wheel, child base_link, origin xyz=-${BASE_LINK_TO_WHEEL_X} 0 ${BASE_LINK_TO_WHEEL_Z} rpy=0 0 0, axis 0 1 0

Commit message: fix(urdf): remove tf_camera argument argument

File: src/bb_description/urdf/beuzebot.urdf (robot description, URDF)
Before this commit: robot beuzebot, 7 links, 5 joints
Joints:
- added joint base_link_to_camera: type fixed, parent base_link, child camera_link, origin xyz=${BASE_LINK_TO_CAMERA_X} ${BASE_LINK_TO_CAMERA_Y} ${BASE_LINK_TO_CAMERA_Z} rpy=${BASE_LINK_TO_CAMERA_ROLL} ${BASE_LINK_TO_CAMERA_PITCH} ${BASE_LINK_TO_CAMERA_YAW}

Commit message: fix(bb_description): set middle_wheel at correct height

File: src/bb_description/urdf/beuzebot.urdf (robot description, URDF)
Before this commit: robot beuzebot, 7 links, 6 joints
Joints:
- joint middle_wheel_to_base: axis 0 1 0 -> (none); origin xyz=-${BASE_LINK_TO_WHEEL_X} 0 ${BASE_LINK_TO_WHEEL_Z} rpy=0 0 0 -> xyz=${-BASE_LINK_TO_WHEEL_X} 0 ${-BASE_LINK_TO_WHEEL_Z} rpy=0 0 0; type continuous -> fixed
